Commit message: casbot

File: src/holosoma_retargeting/holosoma_retargeting/models/casbot/casbot_25dof_spherehand.urdf (robot description, URDF)
Before this commit: robot CB02_URDF(ECS)0801A, 40 links, 39 joints
Links:
- removed link left_hand_link
- removed link right_hand_link
- added link left_sphere_hand_link, mass 0.124; collision mesh filename=../g1/assets/half_sphere.obj; visual mesh filename=../g1/assets/half_sphere.obj
- added link left_sphere_hand_tip_link; collision sphere radius=0.001; visual sphere radius=0.001
- added link right_sphere_hand_link, mass 0.124; collision mesh filename=../g1/assets/half_sphere.obj; visual mesh filename=../g1/assets/half_sphere.obj
- added link right_sphere_hand_tip_link; collision sphere radius=0.001; visual sphere radius=0.001
Joints:
- removed joint left_hand_joint
- removed joint right_hand_joint
- added joint left_hand_palm_joint: type fixed, parent left_wrist_yaw_link, child left_sphere_hand_link, origin xyz=0 0.003 -0.1 rpy=0 3.14159 0
- added joint left_sphere_hand_tip_joint: type fixed, parent left_sphere_hand_link, child left_sphere_hand_tip_link, origin xyz=0.03 0 0 rpy=0 0 0
- added joint right_hand_palm_joint: type fixed, parent right_wrist_yaw_link, child right_sphere_hand_link, origin xyz=0 0.003 -0.1 rpy=0 3.14159 0
- added joint right_sphere_hand_tip_joint: type fixed, parent right_sphere_hand_link, child right_sphere_hand_tip_link, origin xyz=0.03 0 0 rpy=0 0 0

File: src/holosoma_retargeting/holosoma_retargeting/models/casbot_skeleton/casbot_skeleton_25dof.urdf (robot description, URDF)
Before this commit: robot CB02_URDF_ECS_WK_0904B, 26 links, 25 joints
Links:
- added link left_ankle_intermediate_1_link, mass 0.01; collision sphere radius=0.01; visual sphere radius=0.01
- added link left_ankle_roll_sphere_1_link, mass 0.001; collision sphere radius=0.005; visual sphere radius=0.005
- added link left_ankle_roll_sphere_2_link, mass 0.001; collision sphere radius=0.005; visual sphere radius=0.005
- added link left_ankle_roll_sphere_3_link, mass 0.001; collision sphere radius=0.005; visual sphere radius=0.005
- added link left_ankle_roll_sphere_4_link, mass 0.001; collision sphere radius=0.005; visual sphere radius=0.005
- added link left_ankle_roll_sphere_5_link, mass 0.001; collision sphere radius=0.005; visual sphere radius=0.005
- added link right_ankle_intermediate_1_link, mass 0.01; collision sphere radius=0.01; visual sphere radius=0.01
- added link right_ankle_roll_sphere_1_link, mass 0.001; collision sphere radius=0.005; visual sphere radius=0.005
- added link right_ankle_roll_sphere_2_link, mass 0.001; collision sphere radius=0.005; visual sphere radius=0.005
- added link right_ankle_roll_sphere_3_link, mass 0.001; collision sphere radius=0.005; visual sphere radius=0.005
- added link right_ankle_roll_sphere_4_link, mass 0.001; collision sphere radius=0.005; visual sphere radius=0.005
- added link right_ankle_roll_sphere_5_link, mass 0.001; collision sphere radius=0.005; visual sphere radius=0.005
Joints:
- added joint left_ankle_intermediate_1_joint: type fixed, parent left_leg_knee_pitch_link, child left_ankle_intermediate_1_link, origin xyz=0 0 -0.42 rpy=0 0 0
- added joint left_ankle_roll_sphere_1_joint: type fixed, parent left_leg_ankle_roll_link, child left_ankle_roll_sphere_1_link, origin xyz=-0.085 0.045 -0.04 rpy=0 0 0
- added joint left_ankle_roll_sphere_2_joint: type fixed, parent left_leg_ankle_roll_link, child left_ankle_roll_sphere_2_link, origin xyz=-0.085 -0.045 -0.04 rpy=0 0 0
- added joint left_ankle_roll_sphere_3_joint: type fixed, parent left_leg_ankle_roll_link, child left_ankle_roll_sphere_3_link, origin xyz=0.155 0.045 -0.04 rpy=0 0 0
- added joint left_ankle_roll_sphere_4_joint: type fixed, parent left_leg_ankle_roll_link, child left_ankle_roll_sphere_4_link, origin xyz=0.155 -0.045 -0.04 rpy=0 0 0
- added joint left_ankle_roll_sphere_5_joint: type fixed, parent left_leg_ankle_roll_link, child left_ankle_roll_sphere_5_link, origin xyz=0.175 0 -0.04 rpy=0 0 0
- added joint right_ankle_intermediate_1_joint: type fixed, parent right_leg_knee_pitch_link, child right_ankle_intermediate_1_link, origin xyz=0 0 -0.42 rpy=0 0 0
- added joint right_ankle_roll_sphere_1_joint: type fixed, parent right_leg_ankle_roll_link, child right_ankle_roll_sphere_1_link, origin xyz=-0.085 -0.045 -0.04 rpy=0 0 0
- added joint right_ankle_roll_sphere_2_joint: type fixed, parent right_leg_ankle_roll_link, child right_ankle_roll_sphere_2_link, origin xyz=-0.085 0.045 -0.04 rpy=0 0 0
- added joint right_ankle_roll_sphere_3_joint: type fixed, parent right_leg_ankle_roll_link, child right_ankle_roll_sphere_3_link, origin xyz=0.155 -0.045 -0.04 rpy=0 0 0
- added joint right_ankle_roll_sphere_4_joint: type fixed, parent right_leg_ankle_roll_link, child right_ankle_roll_sphere_4_link, origin xyz=0.155 0.045 -0.04 rpy=0 0 0
- added joint right_ankle_roll_sphere_5_joint: type fixed, parent right_leg_ankle_roll_link, child right_ankle_roll_sphere_5_link, origin xyz=0.175 0 -0.04 rpy=0 0 0
